Commit message: Added motor torque constraint handling for all motors

File: cart_pole/my_cartpole.urdf (robot description, URDF)
Before this commit: robot cart_pole, 7 links, 6 joints
Links:
- link cart_base: mass 0.1 -> 0.2

Commit message: Changes

File: cart_pole/my_cartpole.urdf (robot description, URDF)
Before this commit: robot cart_pole, 7 links, 6 joints
Links:
- link mass_link: mass 0.05 -> 0.075
- link pole_link: mass 0.02 -> 0.01
